File: CP_Watsonville_South-Model.sch (EAGLE design)
At the start: 88 parts, among them IC1 MCP23017SO, IC2 MCP23017SO, IC3 MCP23017SO

Commit message: Added 1x6 for MID-model board
Parts:
- added CON1: (no value), SPCoast:CONNECTOR-M06LOCK
Connections:
- new net 1SAAT: CON1.3, IC2.GPB2
- new net 2SAAT: CON1.4, IC2.GPB3
- new net 3SAAT: CON1.5, IC2.GPB4
- new net 4SAAT: CON1.6, IC2.GPB5
- new net DAAT: CON1.2, IC2.GPB1
- net VCC: now also CON1.1
Changed lines of the file:
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@@
 <part name="9NG" library="SPCoast" deviceset="LED*" device="0603-LED" value="G"/>
 <part name="9RR" library="SPCoast" deviceset="LED*" device="0603-LED" value="R"/>
+<part name="CON1" library="SPCoast" deviceset="CONNECTOR-M06" device="LOCK"/>
+<part name="P+19" library="SPCoast" deviceset="VCC" device=""/>
 </parts>
 <sheets>
@@
 <instance part="9NG" gate="LED" x="215.9" y="101.6" rot="R270"/>
 <instance part="9RR" gate="LED" x="228.6" y="101.6" rot="R270"/>
+<instance part="CON1" gate="J" x="99.06" y="91.44" rot="MR180"/>
+<instance part="P+19" gate="VCC" x="104.14" y="99.06"/>
 </instances>
 <busses>
@@
 <wire x1="27.94" y1="35.56" x2="20.32" y2="35.56" width="0.1524" layer="91"/>
 <pinref part="P+18" gate="VCC" pin="VCC"/>
+</segment>
+<segment>
+<pinref part="CON1" gate="J" pin="1"/>
+<pinref part="P+19" gate="VCC" pin="VCC"/>
 </segment>
 </net>
@@
 </segment>
 </net>
+<net name="DAAT" class="0">
+<segment>
+<pinref part="IC2" gate="G$1" pin="GPB1"/>
+<wire x1="53.34" y1="96.52" x2="58.42" y2="96.52" width="0.1524" layer="91"/>
+<label x="58.42" y="96.52" size="1.27" layer="95" xref="yes"/>
+</segment>
+<segment>
+<wire x1="104.14" y1="93.98" x2="109.22" y2="93.98" width="0.1524" layer="91"/>
+<label x="109.22" y="93.98" size="1.27" layer="95" xref="yes"/>
+<pinref part="CON1" gate="J" pin="2"/>
+</segment>
+</net>
+<net name="1SAAT" class="0">
+<segment>
+<pinref part="IC2" gate="G$1" pin="GPB2"/>
+<wire x1="53.34" y1="93.98" x2="58.42" y2="93.98" width="0.1524" layer="91"/>
+<label x="58.42" y="93.98" size="1.27" layer="95" xref="yes"/>
+</segment>
+<segment>
+<wire x1="104.14" y1="91.44" x2="109.22" y2="91.44" width="0.1524" layer="91"/>
+<label x="109.22" y="91.44" size="1.27" layer="95" xref="yes"/>
+<pinref part="CON1" gate="J" pin="3"/>
+</segment>
+</net>
+<net name="2SAAT" class="0">
+<segment>
+<pinref part="IC2" gate="G$1" pin="GPB3"/>
+<wire x1="53.34" y1="91.44" x2="58.42" y2="91.44" width="0.1524" layer="91"/>
+<label x="58.42" y="91.44" size="1.27" layer="95" xref="yes"/>
+</segment>
+<segment>
+<wire x1="104.14" y1="88.9" x2="109.22" y2="88.9" width="0.1524" layer="91"/>
+<label x="109.22" y="88.9" size="1.27" layer="95" xref="yes"/>
+<pinref part="CON1" gate="J" pin="4"/>
+</segment>
+</net>
+<net name="3SAAT" class="0">
+<segment>
+<pinref part="IC2" gate="G$1" pin="GPB4"/>
+<wire x1="53.34" y1="88.9" x2="58.42" y2="88.9" width="0.1524" layer="91"/>
+<label x="58.42" y="88.9" size="1.27" layer="95" xref="yes"/>
+</segment>
+<segment>
+<wire x1="104.14" y1="86.36" x2="109.22" y2="86.36" width="0.1524" layer="91"/>
+<label x="109.22" y="86.36" size="1.27" layer="95" xref="yes"/>
+<pinref part="CON1" gate="J" pin="5"/>
+</segment>
+</net>
+<net name="4SAAT" class="0">
+<segment>
+<pinref part="IC2" gate="G$1" pin="GPB5"/>
+<wire x1="53.34" y1="86.36" x2="58.42" y2="86.36" width="0.1524" layer="91"/>
+<label x="58.42" y="86.36" size="1.27" layer="95" xref="yes"/>
+</segment>
+<segment>
+<wire x1="104.14" y1="83.82" x2="109.22" y2="83.82" width="0.1524" layer="91"/>
+<label x="109.22" y="83.82" size="1.27" layer="95" xref="yes"/>
+<pinref part="CON1" gate="J" pin="6"/>
+</segment>
+</net>
